File: nanoAlt_Alpha/nanoAlt_Alpha.sch (KiCad schematic (older format))
At the start: 10 parts, among them IC1 MS563702BA03-50, J1 AVR_SPI_PROG_3X2TESTPOINTS, U1 ATTINY24A-CCU

Commit message: Fix ERC issues on schematic and update library
Signed-off-by: Pierros Papadeas <pierros@papadeas.gr>
Parts:
- removed U1: ATTINY24A-CCU, My_IC:UFBGA_15CC1, symbol My_IC:ATTINY24A-CCU
- added U1: ATtiny24A-CCU, Package_BGA:UFBGA-15_3.0x3.0mm_Layout4x4_P0.65mm, symbol MCU_Microchip_ATtiny:ATtiny24A-CCU
- C1, C2: value 100nF_0402 -> 100n; footprint My_PASSIVES:0402 -> (none); symbol SparkFun-Capacitors:0.1UF-0603-25V-5% -> Device:C; Field4 CAP-08604 -> (none)
- D1: footprint My_PASSIVES:0402 -> (none)
- IC1: symbol MS563702BA03-50:MS563702BA03-50 -> nanoAlt_Alpha:MS563702BA03-50
- J1: symbol SparkFun-Connectors:AVR_SPI_PROG_3X2TESTPOINTS -> nanoAlt_Alpha:AVR_SPI_PROG_3X2TESTPOINTS-SparkFun-Connectors
- R1, R2, R3: value 10KOHM-0402 -> 10K; footprint My_PASSIVES:0402 -> (none); symbol SparkFun-Resistors:10KOHM-0603-1_10W-1% -> Device:R; Field4 RES-00824 -> (none)
- R4: value 33OHM-0402 -> 33; footprint My_PASSIVES:0402 -> (none); symbol SparkFun-Resistors:33OHM-0603-1_10W-1% -> Device:R; Field4 RES-08270 -> (none)
Connections:
- wire segments 34 -> 39
- no-connect marks 0 -> 7

Commit message: Reroute for 2 layers
Signed-off-by: Pierros Papadeas <pierros@papadeas.gr>
Parts:
- C1, C2: footprint (none) -> Capacitor_SMD:C_0402_1005Metric
- D1: footprint (none) -> LED_SMD:LED_0402_1005Metric
- R1, R2, R3, R4: footprint (none) -> Resistor_SMD:R_0402_1005Metric
Changed lines of the file:
@@
 U 1 1 5B05A2AC
 P 8900 1700
-F 0 "IC1" H 9150 2000 50  0000 L CNN
-F 1 "MS563702BA03-50" H 9150 1900 50  0000 L CNN
+F 0 "IC1" H 9400 1965 50  0000 C CNN
+F 1 "MS563702BA03-50" H 9400 1874 50  0000 C CNN
 F 2 "MS563702BA03-50:MS5637_1" H 9750 1800 50  0001 L CNN
 F 3 "http://docs-europe.electrocomponents.com/webdocs/142c/0900766b8142cddb.pdf" H 9750 1700 50  0001 L CNN
@@
 F 0 "R1" V 7150 3100 45  0000 C CNN
 F 1 "10K" V 7250 3100 45  0000 C CNN
-F 2 "" H 7250 3250 20  0001 C CNN
+F 2 "Resistor_SMD:R_0402_1005Metric" H 7250 3250 20  0001 C CNN
 F 3 "" H 7250 3100 60  0001 C CNN
 F 4 "" H 7250 3300 60  0000 C CNN "Field4"
@@
 F 0 "C1" H 5150 1750 45  0000 L BNN
 F 1 "100n" H 5100 1650 45  0000 L BNN
-F 2 "" H 5400 1950 20  0001 C CNN
+F 2 "Capacitor_SMD:C_0402_1005Metric" H 5400 1950 20  0001 C CNN
 F 3 "" H 5400 1700 50  0001 C CNN
 F 4 "" H 5100 1850 60  0000 C CNN "Field4"
@@
 F 0 "C2" H 8700 2100 45  0000 L BNN
 F 1 "100n" H 8700 2000 45  0000 L BNN
-F 2 "" H 8600 2300 20  0001 C CNN
+F 2 "Capacitor_SMD:C_0402_1005Metric" H 8600 2300 20  0001 C CNN
 F 3 "" H 8600 2050 50  0001 C CNN
 F 4 "" H 8300 2200 60  0000 C CNN "Field4"
@@
 U 1 1 5B05B385
 P 6400 4600
-F 0 "J1" H 6200 4800 45  0000 L BNN
-F 1 "AVR_SPI_PROG_3X2TESTPOINTS" H 5700 4350 45  0000 L BNN
+F 0 "J1" H 6400 4904 45  0000 C CNN
+F 1 "AVR_SPI_PROG_3X2TESTPOINTS" H 6400 4820 45  0000 C CNN
 F 2 "My_Connectors:50mil_POGO" H 6400 4900 20  0001 C CNN
 F 3 "" H 6400 4600 50  0001 C CNN
@@
 F 0 "R2" V 9050 3650 45  0000 C CNN
 F 1 "10K" V 8950 3650 45  0000 C CNN
-F 2 "" H 8950 3800 20  0001 C CNN
+F 2 "Resistor_SMD:R_0402_1005Metric" H 8950 3800 20  0001 C CNN
 F 3 "" H 8950 3650 60  0001 C CNN
 F 4 "" H 8950 3800 60  0000 C CNN "Field4"
@@
 F 0 "R3" V 9050 3350 45  0000 C CNN
 F 1 "10K" V 8950 3350 45  0000 C CNN
-F 2 "" H 8950 3500 20  0001 C CNN
+F 2 "Resistor_SMD:R_0402_1005Metric" H 8950 3500 20  0001 C CNN
 F 3 "" H 8950 3350 60  0001 C CNN
 F 4 "" H 8950 3500 60  0000 C CNN "Field4"
@@
 F 0 "R4" V 7200 1900 45  0000 C CNN
 F 1 "33" V 7100 1900 45  0000 C CNN
-F 2 "" H 7100 2050 20  0001 C CNN
+F 2 "Resistor_SMD:R_0402_1005Metric" H 7100 2050 20  0001 C CNN
 F 3 "" H 7100 1900 60  0001 C CNN
 F 4 "" H 7100 2100 60  0000 C CNN "Field4"
@@
 F 0 "D1" H 7500 2000 50  0000 C CNN
 F 1 "LED" H 7500 1800 50  0000 C CNN
-F 2 "" H 7500 1900 50  0001 C CNN
+F 2 "LED_SMD:LED_0402_1005Metric" H 7500 1900 50  0001 C CNN
 F 3 "" H 7500 1900 50  0001 C CNN
 	1    7500 1900
